Commit message: Gazebo: massa corpo realistica + baricentro spostato indietro (Pi posteriore)
Geometria confermata corretta dall'utente (spaziatura swing 165mm uniforme, le
zampe cadono a distanze diverse per l'offset FWD invertito dietro: gia' modellato).
Sistemo la MASSA: BODY_MASS 0.6->0.75 e COM del corpo 45mm dietro il centro
(Raspberry sulla fila posteriore) -> baricentro come nel robot vero. Totale ~1.3kg.
Approssimazione: si raffina con una misura reale del COM.

Co-Authored-By: Claude Opus 4.8 (1M context) <noreply@anthropic.com>

File: description/genghis_gazebo.urdf (robot description, URDF)
Before this commit: robot genghis, 22 links, 21 joints
Links:
- link base_link: mass 0.6 -> 0.75
